Commit message: second

File: chapter05/baxter_camera/urdf/baxter_base/baxter_base_camera.urdf.xacro (robot description, xacro)
@@ -30,5 +30,5 @@
     </inertial>
   </link>
-  <!--link name="RGBD_camera">
+  <link name="RGBD_camera">
     <visual>
        <origin xyz="0.0 0.0 0" rpy="0.0 0.0 0.0"/>
@@ -37,5 +37,5 @@
        </geometry>
     </visual>
-  </link-->
+  </link>
   <link name="left_torso_itb">
     <inertial>
@@ -213,9 +213,9 @@
     <limit effort="50000" lower="-3.01" upper="3.01" velocity="10000"/>
   </joint>
-  <!--joint name="RGBD_camera_joint" type="fixed">
+  <joint name="RGBD_camera_joint" type="fixed">
     <origin rpy="0 ${pi/9} 0" xyz="0.06 0 0.96"/>
     <parent link="torso"/>
     <child link="RGBD_camera"/>
-  </joint-->
+  </joint>
   <joint name="left_torso_itb_fixed" type="fixed">
     <origin rpy="-1.57079632679 3.1415 0" xyz="-0.08897 0.15593 0.389125"/>
