Commit message: baxter_success

File: chapter05/baxter_camera/urdf/baxter_base/baxter_base_kinect.gazebo.xacro (robot description, xacro)
@@ -92,5 +92,5 @@
         <cameraInfoTopicName>camera_info</cameraInfoTopicName>
         <depthImageCameraInfoTopicName>camera_info</depthImageCameraInfoTopicName>
-        <frameName>kinect</frameName>
+        <frameName>kinect_optical_frame</frameName>
         <baseline>0.1</baseline>
         <distortion_k1>-0.11862627596824302</distortion_k1>

File: chapter05/baxter_camera/urdf/baxter_base/baxter_base_kinect.urdf.xacro (robot description, xacro)
@@ -35,5 +35,5 @@
             <color rgba="0.1 0.1 0.1 1.0"/>
         </material>
-       <origin xyz="0.0 0.0 0" rpy="0.0 0 0.0"/>
+       <origin xyz="-0.05 0.0 -0.03" rpy="${-pi} ${pi} ${pi}"/>
        <geometry>
          <mesh filename="package://baxter_camera/meshes/kinectv2/kinectv2.stl"/>
@@ -41,5 +41,5 @@
     </visual>
     <collision>
-      <origin xyz="0.0 0.0 0.0" rpy="0 0 0"/>
+      <origin xyz="-0.05 0.0 -0.03" rpy="${-pi} ${pi} ${pi}"/>
       <geometry>
         <mesh filename="package://baxter_camera/meshes/kinectv2/kinectv2.stl"/>
@@ -225,5 +225,5 @@
 <!-- You can Change    -->
   <joint name="kinect_joint" type="fixed">
-    <origin  xyz="0.09 0 0.88" rpy="0 0 0"/>
+    <origin  xyz="0.15 0 0.88" rpy="0 ${pi/8} 0"/>
     <parent link="torso"/>
     <child link="kinect"/>

File: chapter05/baxter_camera/urdf/baxter_kinect.urdf.xacro (robot description, xacro)
@@ -6,4 +6,10 @@
   </xacro:include>
   <xacro:include filename="$(find baxter_camera)/urdf/baxter_base/baxter_base_kinect.gazebo.xacro"></xacro:include>
+  <link name="kinect_optical_frame"/>
+  <joint name="kinect_optical_joint" type="fixed">
+    <parent link="torso"/>
+    <child link="kinect_optical_frame"/>
+    <origin  xyz="0.15 0 0.88" rpy="${41*pi/30} 0 ${-pi/2}"/>
+  </joint>
   <!-- Baxter Pedestal -->
   <xacro:if value="$(arg pedestal)">
