Commit message: gazebo_seikou

File: chapter05/baxter_camera/urdf/baxter.urdf (robot description, URDF)
Before this commit: robot baxter, 49 links, 48 joints
Links:
- link head: geometry collision sphere radius=0.001; visual mesh filename=package://baxter_camera/meshes/head/H0.DAE
- link left_lower_elbow: geometry collision cylinder length=0.10 radius=0.06; visual mesh filename=package://baxter_camera/meshes/lower_elbow/E1.DAE
- link left_lower_forearm: geometry collision cylinder length=0.10 radius=0.06; visual mesh filename=package://baxter_camera/meshes/lower_forearm/W1.DAE
- link left_lower_shoulder: geometry collision cylinder length=0.12 radius=0.06; visual mesh filename=package://baxter_camera/meshes/lower_shoulder/S1.DAE
- link left_upper_elbow: geometry collision cylinder length=0.107 radius=0.06; visual mesh filename=package://baxter_camera/meshes/upper_elbow/E0.DAE
- link left_upper_forearm: geometry collision cylinder length=0.088 radius=0.06; visual mesh filename=package://baxter_camera/meshes/upper_forearm/W0.DAE
- link left_upper_shoulder: geometry collision cylinder length=0.2722 radius=0.06; visual mesh filename=package://baxter_camera/meshes/upper_shoulder/S0.DAE
- link left_wrist: geometry collision cylinder length=0.165 radius=0.06; visual mesh filename=package://baxter_camera/meshes/wrist/W2.DAE
- link pedestal: geometry collision mesh filename=package://baxter_camera/meshes/base/pedestal_link_collision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; visual mesh filename=package://baxter_camera/meshes/base/PEDESTAL.DAE
- link right_lower_elbow: geometry collision cylinder length=0.10 radius=0.06; visual mesh filename=package://baxter_camera/meshes/lower_elbow/E1.DAE
- link right_lower_forearm: geometry collision cylinder length=0.10 radius=0.06; visual mesh filename=package://baxter_camera/meshes/lower_forearm/W1.DAE
- link right_lower_shoulder: geometry collision cylinder length=0.12 radius=0.06; visual mesh filename=package://baxter_camera/meshes/lower_shoulder/S1.DAE
- link right_upper_elbow: geometry collision cylinder length=0.107 radius=0.06; visual mesh filename=package://baxter_camera/meshes/upper_elbow/E0.DAE
- link right_upper_forearm: geometry collision cylinder length=0.088 radius=0.06; visual mesh filename=package://baxter_camera/meshes/upper_forearm/W0.DAE
- link right_upper_shoulder: geometry collision cylinder length=0.2722 radius=0.06; visual mesh filename=package://baxter_camera/meshes/upper_shoulder/S0.DAE
- link right_wrist: geometry collision cylinder length=0.165 radius=0.06; visual mesh filename=package://baxter_camera/meshes/wrist/W2.DAE
- link screen: geometry collision sphere radius=0.001; visual mesh filename=package://baxter_camera/meshes/head/H1.DAE
- link torso: geometry collision mesh filename=package://baxter_camera/meshes/torso/base_link_collision.DAE; visual mesh filename=package://baxter_camera/meshes/torso/base_link.DAE

File: chapter05/baxter_camera/urdf/baxter_base/baxter_base_kinect.urdf.xacro (robot description, xacro)
@@ -1,9 +1,4 @@
 <?xml version="1.0" ?>
 <robot name="baxter" xmlns:xacro="http://www.ros.org/wiki/xacro">
-  <xacro:arg name="gazebo" default="false"/>
-  <xacro:if value="$(arg gazebo)">
-    <!-- Gazebo Tags -->
-    <xacro:include filename="$(find baxter_camera)/urdf/baxter_base/baxter_base.gazebo.xacro" />
-  </xacro:if>
   <link name="base">
   </link>
@@ -31,13 +26,24 @@
   </link>
   <link name="kinect">
+    <inertial>
+      <origin rpy="0 0 0" xyz="0.000000 0.000000 0.000000"/>
+      <mass value="0.0001"/>
+      <inertia ixx="1e-08" ixy="0" ixz="0" iyy="1e-08" iyz="0" izz="1e-08"/>
+    </inertial>
     <visual>
         <material name="black">
             <color rgba="0.1 0.1 0.1 1.0"/>
         </material>
-       <origin xyz="0.0 0.0 0" rpy="0.0 0.0 0.0"/>
+       <origin xyz="0.0 0.0 0" rpy="0.0 ${-pi/4} 0.0"/>
        <geometry>
          <mesh filename="package://baxter_camera/meshes/kinectv2/kinectv2.stl"/>
        </geometry>
     </visual>
+    <collision>
+      <origin rpy="0 ${-pi/4} 0" xyz="0.0 0.0 0.0"/>
+      <geometry>
+        <mesh filename="package://baxter_camera/meshes/kinectv2/kinectv2.stl"/>
+      </geometry>
+    </collision>
   </link>
   <link name="left_torso_itb">
@@ -217,5 +223,5 @@
   </joint>
   <joint name="kinect_joint" type="fixed">
-    <origin rpy="0 ${pi/9} 0" xyz="0.09 0 0.88"/>
+    <origin rpy="${3*pi/4} ${3*pi/18} 0" xyz="0.09 0 0.88"/>
     <parent link="torso"/>
     <child link="kinect"/>

File: chapter05/baxter_camera/urdf/baxter_kinect.urdf.xacro (robot description, xacro)
@@ -1,10 +1,9 @@
 <?xml version="1.0" ?>
 <robot name="baxter" xmlns:xacro="http://www.ros.org/wiki/xacro">
-  <xacro:arg name="gazebo" default="false"/>
   <xacro:arg name="pedestal" default="true"/>
   <!-- Baxter Base URDF -->
   <xacro:include filename="$(find baxter_camera)/urdf/baxter_base/baxter_base_kinect.urdf.xacro">
-    <xacro:arg name="gazebo" value="${gazebo}"/>
   </xacro:include>
+  <xacro:include filename="$(find baxter_camera)/urdf/baxter_base/baxter_base_kinect.gazebo.xacro"></xacro:include>
   <!-- Baxter Pedestal -->
   <xacro:if value="$(arg pedestal)">

File: chapter05/baxter_camera/urdf/pedestal/pedestal.xacro (robot description, xacro)
@@ -7,5 +7,5 @@
       <origin rpy="0 0 0" xyz="0 0 0"/>
       <geometry>
-        <mesh filename="package://baxter_description/meshes/base/PEDESTAL.DAE"/>
+        <mesh filename="package://baxter_camera/meshes/base/PEDESTAL.DAE"/>
       </geometry>
       <material name="darkgray">
@@ -16,5 +16,5 @@
       <origin rpy="0 0 0" xyz="0 0 0"/>
       <geometry>
-        <mesh filename="package://baxter_description/meshes/base/pedestal_link_collision.DAE"/>
+        <mesh filename="package://baxter_camera/meshes/base/pedestal_link_collision.DAE"/>
       </geometry>
     </collision>
