Commit message: senco

File: chapter06/baxter_camera/urdf/baxter_base/baxter_base_kinect.gazebo.xacro (robot description, xacro)
@@ -337,4 +337,42 @@
     </plugin>
   </gazebo>
+  <gazebo>
+    <plugin name="gazebo_grasp_fix_right" filename="libgazebo_grasp_fix.so">
+      <arm>
+        <arm_name>baxter_right</arm_name>
+        <palm_link>right_wrist</palm_link>
+        <gripper_link>r_gripper_l_finger</gripper_link>
+        <gripper_link>r_gripper_r_finger</gripper_link>
+      </arm>
+      <arm>
+        <arm_name>baxter_left</arm_name>
+        <palm_link>left_wrist</palm_link>
+        <gripper_link>l_gripper_l_finger</gripper_link>
+        <gripper_link>l_gripper_r_finger</gripper_link>
+      </arm>
+      <forces_angle_tolerance>100</forces_angle_tolerance>
+			<update_rate>4</update_rate>
+			<grip_count_threshold>4</grip_count_threshold>
+			<max_grip_count>8</max_grip_count>
+			<release_tolerance>0.02</release_tolerance>
+			<disable_collisions_on_attach>false</disable_collisions_on_attach>
+			<contact_topic>__default_topic__right</contact_topic>
+    </plugin>
+    <!--plugin name="gaebo_grasp_fix_left" filename="libgazebo_grasp_fix.so">
+      <arm>
+        <arm_name>baxter_left</arm_name>
+        <palm_link>left_wrist</palm_link>
+        <gripper_link>l_gripper_l_finger</gripper_link>
+        <gripper_link>l_gripper_r_finger</gripper_link>
+      </arm>
+      <forces_angle_tolerance>100</forces_angle_tolerance>
+			<update_rate>4</update_rate>
+			<grip_count_threshold>4</grip_count_threshold>
+			<max_grip_count>8</max_grip_count>
+			<release_tolerance>0.005</release_tolerance>
+			<disable_collisions_on_attach>false</disable_collisions_on_attach>
+			<contact_topic>__default_topic__left</contact_topic>
+    </plugin-->
+  </gazebo>
   <!-- Transmissions -->
   <!-- Right Arm -->

File: chapter06/baxter_camera/urdf/baxter_base/baxter_base_kinect.urdf.xacro (robot description, xacro)
@@ -16,5 +16,5 @@
       <origin rpy="0 0 0" xyz="0 0 0"/>
       <geometry>
-        <mesh filename="package://baxter_camera/meshes/torso/base_link_collision.DAE"/>
+        <mesh filename="package://baxter_camera/meshes/torso/base_link.STL"/>
       </geometry>
     </collision>
@@ -75,5 +75,5 @@
       <origin rpy="0 0 0" xyz="0.0 0 0.0"/>
       <geometry>
-        <sphere radius="0.001"/>
+        <mesh filename="package://baxter_camera/meshes/head/H0.STL"/>
       </geometry>
     </collision>
@@ -119,5 +119,5 @@
       <origin rpy="0 0 0" xyz="0.0 0 0.0"/>
       <geometry>
-        <sphere radius="0.001"/>
+        <mesh filename="package://baxter_camera/meshes/head/H1.STL"/>
       </geometry>
     </collision>
@@ -289,5 +289,5 @@
       <origin rpy="0 0 0" xyz="0 0 0.1361"/>
       <geometry>
-        <cylinder length="0.2722" radius="0.06"/>
+        <mesh filename="package://baxter_camera/meshes/upper_shoulder/S0.STL"/>
       </geometry>
     </collision>

File: chapter06/baxter_camera/urdf/electric_gripper/fingers/extended_narrow.xacro (robot description, xacro)
@@ -15,10 +15,10 @@
       <xacro:property name="finger_box_length" value="0.0615" scope="local"/>
       <collision>
-        <origin rpy="0 0 ${-pi/2*(reflect+1)}" xyz="0 ${finger_width*reflect} ${finger_box_length}"/>
+        <origin rpy="0 0 ${-pi/2*(reflect+1)}" xyz="0 0 0"/>
         <geometry>
-          <box size="${finger_box_height} ${finger_box_width} ${finger_length}"/>
+          <mesh filename="package://baxter_camera/meshes/electric_gripper/fingers/extended_narrow.STL" />
         </geometry>
       </collision>
-      <xacro:property name="knuckle_box_height" value="0.01" scope="local"/>
+      <!--xacro:property name="knuckle_box_height" value="0.01" scope="local"/>
       <xacro:property name="knuckle_box_width" value="0.017" scope="local"/>
       <xacro:property name="knuckle_box_length" value="${finger_width + 0.03275}" scope="local"/>
@@ -28,5 +28,5 @@
           <box size="${knuckle_box_height} ${knuckle_box_length} ${knuckle_box_width}"/>
         </geometry>
-      </collision>
+      </collision-->
       <inertial>
         <origin rpy="0 0 ${-pi/2*(reflect+1)}" xyz="0 0 0"/>

File: chapter06/baxter_camera/urdf/electric_gripper/fingers/half_round_tip.xacro (robot description, xacro)
@@ -16,5 +16,5 @@
         <origin rpy="0 0 ${pi*(g_reflect+1)/2}" xyz="0 ${-0.0045*g_reflect} -0.015"/>
         <geometry>
-          <cylinder length="0.037" radius="0.008"/>
+          <mesh filename="package://baxter_camera/meshes/electric_gripper/fingers/half_round_tip.DAE" />
         </geometry>
       </collision>

File: chapter06/baxter_camera/urdf/electric_gripper/fingers/paddle_tip.xacro (robot description, xacro)
@@ -16,5 +16,5 @@
         <origin rpy="0 0 ${pi*(g_reflect+1)/2}" xyz="0 ${-0.0045*g_reflect} -0.015"/>
         <geometry>
-          <box size="0.042 0.0065 0.037"/>
+          <mesh filename="package://baxter_camera/meshes/electric_gripper/fingers/paddle_tip.STL" />
         </geometry>
       </collision>

File: chapter06/baxter_camera/urdf/electric_gripper/rethink_electric_gripper.xacro (robot description, xacro)
@@ -14,5 +14,5 @@
         <origin rpy="${-pi/2} ${pi} 0" xyz="0.0 0.0 0"/>
         <geometry>
-          <cylinder length="0.1" radius="0.029"/>
+          <mesh filename="package://baxter_camera/meshes/electric_gripper/electric_gripper_base.DAE"/>
         </geometry>
         <material name="darkred">
@@ -78,5 +78,5 @@
       <dynamics damping="0.7" friction="0.0"/>
     </joint>
-    <transmission name="gripper_${side}1">
+    <!--transmission name="gripper_${side}1">
       <type>transmission_interface/SimpleTransmission</type>
       <joint name="${gripper_side}_gripper_r_finger_joint">
@@ -87,5 +87,5 @@
         <mechanicalReduction>1</mechanicalReduction>
       </actuator>
-    </transmission>
+    </transmission-->
     <transmission name="gripper_${side}2">
       <type>transmission_interface/SimpleTransmission</type>
@@ -94,5 +94,5 @@
       </joint>
       <actuator name="gripper_${gripper_side}1_motor2">
-        <!--hardwareInterface>hardware_interface/PositionJointInterface</hardwareInterface-->
+        <hardwareInterface>hardware_interface/PositionJointInterface</hardwareInterface>
         <mechanicalReduction>1</mechanicalReduction>
       </actuator>

Commit message: sefond

File: chapter06/baxter_camera/urdf/baxter_base/baxter_base_kinect.gazebo.xacro (robot description, xacro)
@@ -4,7 +4,7 @@
   <!-- ros_control plugin -->
   <gazebo>
-    <plugin name="baxter_ros_control" filename="libbaxter_gazebo_ros_control.so">
+    <!--plugin name="baxter_ros_control" filename="libbaxter_gazebo_ros_control.so">
       <robotNamespace>/robot</robotNamespace>
-    </plugin>
+    </plugin-->
   </gazebo>
   <!-- Gazebo-Specific Link Properties -->
@@ -327,11 +327,11 @@
   <gazebo>
     <plugin name="mimic_joint_plugin_left" filename="libroboticsgroup_gazebo_mimic_joint_plugin.so">
-      <joint>l_gripper_l_finger_joint</joint>
-      <mimicJoint>l_gripper_r_finger_joint</mimicJoint>
+      <joint>l_gripper_l_finger_joint_1</joint>
+      <mimicJoint>l_gripper_r_finger_joint_1</mimicJoint>
       <multiplier>-1.0</multiplier>
     </plugin>
     <plugin name="mimic_joint_plugin_right" filename="libroboticsgroup_gazebo_mimic_joint_plugin.so">
-      <joint>r_gripper_l_finger_joint</joint>
-      <mimicJoint>r_gripper_r_finger_joint</mimicJoint>
+      <joint>r_gripper_l_finger_joint_1</joint>
+      <mimicJoint>r_gripper_r_finger_joint_1</mimicJoint>
       <multiplier>-1.0</multiplier>
     </plugin>
@@ -339,10 +339,10 @@
   <gazebo>
     <plugin name="gazebo_grasp_fix_right" filename="libgazebo_grasp_fix.so">
-      <arm>
+      <!--arm>
         <arm_name>baxter_right</arm_name>
         <palm_link>right_wrist</palm_link>
         <gripper_link>r_gripper_l_finger</gripper_link>
         <gripper_link>r_gripper_r_finger</gripper_link>
-      </arm>
+      </arm-->
       <arm>
         <arm_name>baxter_left</arm_name>
@@ -355,7 +355,7 @@
 			<grip_count_threshold>4</grip_count_threshold>
 			<max_grip_count>8</max_grip_count>
-			<release_tolerance>0.02</release_tolerance>
+			<release_tolerance>0.001</release_tolerance>
 			<disable_collisions_on_attach>false</disable_collisions_on_attach>
-			<contact_topic>__default_topic__right</contact_topic>
+			<contact_topic>__default_topic__</contact_topic>
     </plugin>
     <!--plugin name="gaebo_grasp_fix_left" filename="libgazebo_grasp_fix.so">

File: chapter06/baxter_camera/urdf/baxter_base/baxter_base_kinect.urdf.xacro (robot description, xacro)
@@ -143,4 +143,13 @@
       <inertia ixx="1e-08" ixy="0" ixz="0" iyy="1e-08" iyz="0" izz="1e-08"/>
     </inertial>
+    <collision>
+      <origin rpy="0.2617993877991494 0 0" xyz="0 0 0"/>
+      <geometry>
+        <box size="0.218 0.16 0.001"/>
+      </geometry>
+      <material name="black">
+        <color rgba="0 0 0 1"/>
+      </material>
+    </collision>
   </link>
   <link name="head_camera">
@@ -203,11 +212,11 @@
   </link>
   <joint name="collision_head_1" type="fixed">
-    <origin rpy="0 0 0" xyz="0.11 0 0.75"/>
-    <parent link="base"/>
+    <origin rpy="0 0 0" xyz="0.11 0 1.68"/>
+    <parent link="pedestal"/>
     <child link="collision_head_link_1"/>
   </joint>
   <joint name="collision_head_2" type="fixed">
-    <origin rpy="0 0 0" xyz="0.11 0 0.75"/>
-    <parent link="base"/>
+    <origin rpy="0 0 0" xyz="0.11 0 1.68"/>
+    <parent link="pedestal"/>
     <child link="collision_head_link_2"/>
   </joint>
@@ -218,6 +227,6 @@
   </joint>
   <joint name="torso_t0" type="fixed">
-    <origin rpy="0 0 0" xyz="0 0 0"/>
-    <parent link="base"/>
+    <origin rpy="0 0 0" xyz="0 0 0.93"/>
+    <parent link="pedestal"/>
     <child link="torso"/>
     <limit effort="50000" lower="-3.01" upper="3.01" velocity="10000"/>
@@ -491,27 +500,45 @@
       <inertia ixx="1e-08" ixy="0" ixz="0" iyy="1e-08" iyz="0" izz="1e-08"/>
     </inertial>
-  </link>
-  <link name="right_hand_camera_axis">
-    <inertial>
-      <origin rpy="0 0 0" xyz="0 0 0"/>
-      <mass value="0.0001"/>
-      <inertia ixx="1e-08" ixy="0" ixz="0" iyy="1e-08" iyz="0" izz="1e-08"/>
-    </inertial>
-  </link>
-  <link name="right_hand_range">
-    <visual>
-      <origin rpy="0 0 0" xyz="0 0 0"/>
-      <geometry>
-        <box size="0.005 .02 .005"/>
+    <collision>
+      <origin rpy="0 0 0" xyz="0 0 0"/>
+      <geometry>
+        <cylinder length="0.01" radius="0.02"/>
       </geometry>
       <material name="blue">
         <color rgba="0 0 1 0.8"/>
       </material>
-    </visual>
-    <inertial>
-      <origin rpy="0 0 0" xyz="0 0 0"/>
-      <mass value="0.0001"/>
-      <inertia ixx="1e-08" ixy="0" ixz="0" iyy="1e-08" iyz="0" izz="1e-08"/>
-    </inertial>
+    </collision>
+  </link>
+  <link name="right_hand_camera_axis">
+    <inertial>
+      <origin rpy="0 0 0" xyz="0 0 0"/>
+      <mass value="0.0001"/>
+      <inertia ixx="1e-08" ixy="0" ixz="0" iyy="1e-08" iyz="0" izz="1e-08"/>
+    </inertial>
+  </link>
+  <link name="right_hand_range">
+    <visual>
+      <origin rpy="0 0 0" xyz="0 0 0"/>
+      <geometry>
+        <box size="0.005 .02 .005"/>
+      </geometry>
+      <material name="blue">
+        <color rgba="0 0 1 0.8"/>
+      </material>
+    </visual>
+    <inertial>
+      <origin rpy="0 0 0" xyz="0 0 0"/>
+      <mass value="0.0001"/>
+      <inertia ixx="1e-08" ixy="0" ixz="0" iyy="1e-08" iyz="0" izz="1e-08"/>
+    </inertial>
+    <collision>
+      <origin rpy="0 0 0" xyz="0 0 0"/>
+      <geometry>
+        <box size="0.005 .02 .005"/>
+      </geometry>
+      <material name="blue">
+        <color rgba="0 0 1 0.8"/>
+      </material>
+    </collision>
   </link>
   <link name="right_hand_accelerometer">
@@ -530,4 +557,13 @@
       <inertia ixx="1e-08" ixy="0" ixz="0" iyy="1e-08" iyz="0" izz="1e-08"/>
     </inertial>
+    <collision>
+      <origin rpy="0 0 0" xyz="0 0 0"/>
+      <geometry>
+        <box size="0.01 0.01 0.01"/>
+      </geometry>
+      <material name="black">
+        <color rgba="0 0 0 1"/>
+      </material>
+    </collision>
   </link>
   <joint name="right_torso_arm_mount" type="fixed">
@@ -859,27 +895,45 @@
       <inertia ixx="1e-08" ixy="0" ixz="0" iyy="1e-08" iyz="0" izz="1e-08"/>
     </inertial>
-  </link>
-  <link name="left_hand_camera_axis">
-    <inertial>
-      <origin rpy="0 0 0" xyz="0 0 0"/>
-      <mass value="0.0001"/>
-      <inertia ixx="1e-08" ixy="0" ixz="0" iyy="1e-08" iyz="0" izz="1e-08"/>
-    </inertial>
-  </link>
-  <link name="left_hand_range">
-    <visual>
-      <origin rpy="0 0 0" xyz="0 0 0"/>
-      <geometry>
-        <box size="0.005 .02 .005"/>
+    <collision>
+      <origin rpy="0 0 0" xyz="0 0 0"/>
+      <geometry>
+        <cylinder length="0.01" radius="0.02"/>
       </geometry>
       <material name="blue">
         <color rgba="0 0 1 0.8"/>
       </material>
-    </visual>
-    <inertial>
-      <origin rpy="0 0 0" xyz="0 0 0"/>
-      <mass value="0.0001"/>
-      <inertia ixx="1e-08" ixy="0" ixz="0" iyy="1e-08" iyz="0" izz="1e-08"/>
-    </inertial>
+    </collision>
+  </link>
+  <link name="left_hand_camera_axis">
+    <inertial>
+      <origin rpy="0 0 0" xyz="0 0 0"/>
+      <mass value="0.0001"/>
+      <inertia ixx="1e-08" ixy="0" ixz="0" iyy="1e-08" iyz="0" izz="1e-08"/>
+    </inertial>
+  </link>
+  <link name="left_hand_range">
+    <visual>
+      <origin rpy="0 0 0" xyz="0 0 0"/>
+      <geometry>
+        <box size="0.005 .02 .005"/>
+      </geometry>
+      <material name="blue">
+        <color rgba="0 0 1 0.8"/>
+      </material>
+    </visual>
+    <inertial>
+      <origin rpy="0 0 0" xyz="0 0 0"/>
+      <mass value="0.0001"/>
+      <inertia ixx="1e-08" ixy="0" ixz="0" iyy="1e-08" iyz="0" izz="1e-08"/>
+    </inertial>
+    <collision>
+      <origin rpy="0 0 0" xyz="0 0 0"/>
+      <geometry>
+        <box size="0.005 .02 .005"/>
+      </geometry>
+      <material name="blue">
+        <color rgba="0 0 1 0.8"/>
+      </material>
+    </collision>
   </link>
   <link name="left_hand_accelerometer">
@@ -898,4 +952,13 @@
       <inertia ixx="1e-08" ixy="0" ixz="0" iyy="1e-08" iyz="0" izz="1e-08"/>
     </inertial>
+    <collision>
+      <origin rpy="0 0 0" xyz="0 0 0"/>
+      <geometry>
+        <box size="0.01 0.01 0.01"/>
+      </geometry>
+      <material name="black">
+        <color rgba="0 0 0 1"/>
+      </material>
+    </collision>
   </link>
   <joint name="left_torso_arm_mount" type="fixed">

File: chapter06/baxter_camera/urdf/baxter_kinect.urdf.xacro (robot description, xacro)
@@ -1,6 +1,5 @@
 <?xml version="1.0" ?>
 <robot name="baxter" xmlns:xacro="http://www.ros.org/wiki/xacro">
-  <xacro:arg name="gazebo" default="true"/>
-  <xacro:arg name="pedestal" default="true"/>
+  <xacro:include filename="$(find baxter_camera)/urdf/pedestal/pedestal.xacro"/>
   <!-- Baxter Base URDF -->
   <xacro:include filename="$(find baxter_camera)/urdf/baxter_base/baxter_base_kinect.urdf.xacro">
@@ -14,9 +13,4 @@
   </joint>
   <!-- Baxter Pedestal -->
-  <xacro:if value="$(arg pedestal)">
-    <xacro:include filename="$(find baxter_camera)/urdf/pedestal/pedestal.xacro">
-      <xacro:arg name="gazebo" value="${gazebo}"/>
-    </xacro:include>
-  </xacro:if>
   <!-- Left End Effector -->
   <xacro:include filename="$(find baxter_camera)/urdf/left_end_effector.urdf.xacro" />

File: chapter06/baxter_camera/urdf/electric_gripper/fingers/half_round_tip.xacro (robot description, xacro)
@@ -16,5 +16,5 @@
         <origin rpy="0 0 ${pi*(g_reflect+1)/2}" xyz="0 ${-0.0045*g_reflect} -0.015"/>
         <geometry>
-          <mesh filename="package://baxter_camera/meshes/electric_gripper/fingers/half_round_tip.DAE" />
+          <mesh filename="package://baxter_camera/meshes/electric_gripper/fingers/half_round_tip.STL" />
         </geometry>
       </collision>

File: chapter06/baxter_camera/urdf/electric_gripper/rethink_electric_gripper.xacro (robot description, xacro)
@@ -14,5 +14,5 @@
         <origin rpy="${-pi/2} ${pi} 0" xyz="0.0 0.0 0"/>
         <geometry>
-          <mesh filename="package://baxter_camera/meshes/electric_gripper/electric_gripper_base.DAE"/>
+          <mesh filename="package://baxter_camera/meshes/electric_gripper/electric_gripper_base.STL"/>
         </geometry>
         <material name="darkred">
@@ -59,5 +59,5 @@
     <!-- Left finger -->
     <xacro:property name="l_finger_offset" value="${((l_finger_slot-1)*0.0095) -0.011}" scope="local"/>
-    <joint name="${gripper_side}_gripper_l_finger_joint" type="prismatic">
+    <joint name="${gripper_side}_gripper_l_finger_joint_1" type="prismatic">
       <origin rpy="0 0 0" xyz="0.0 ${l_finger_offset} 0.02"/>
       <axis xyz="0 1 0"/>
@@ -69,5 +69,5 @@
     <!-- Right finger -->
     <xacro:property name="r_finger_offset" value="${((r_finger_slot-1)*-0.0095) +0.011}" scope="local"/>
-    <joint name="${gripper_side}_gripper_r_finger_joint" type="prismatic">
+    <joint name="${gripper_side}_gripper_r_finger_joint_1" type="prismatic">
       <origin rpy="0 0 0" xyz="0.0 ${r_finger_offset} 0.02"/>
       <axis xyz="0 1 0"/>
@@ -75,5 +75,5 @@
       <child link="${gripper_side}_gripper_r_finger"/>
       <limit effort="20.0" lower="-0.020833" upper="0.0" velocity="0.15"/>
-      <mimic joint="${gripper_side}_gripper_l_finger_joint" multiplier="-1.0"/>
+      <mimic joint="${gripper_side}_gripper_l_finger_joint_1" multiplier="-1.0"/>
       <dynamics damping="0.7" friction="0.0"/>
     </joint>
@@ -90,5 +90,5 @@
     <transmission name="gripper_${side}2">
       <type>transmission_interface/SimpleTransmission</type>
-      <joint name="${gripper_side}_gripper_l_finger_joint">
+      <joint name="${gripper_side}_gripper_l_finger_joint_1">
         <hardwareInterface>hardware_interface/PositionJointInterface</hardwareInterface>
       </joint>
@@ -98,8 +98,8 @@
       </actuator>
     </transmission>
-    <gazebo reference="${gripper_side}_gripper_r_finger_joint">
+    <gazebo reference="${gripper_side}_gripper_r_finger_joint_1">
       <implicitSpringDamper>1</implicitSpringDamper>
     </gazebo>
-    <gazebo reference="${gripper_side}_gripper_l_finger_joint">
+    <gazebo reference="${gripper_side}_gripper_l_finger_joint_1">
       <implicitSpringDamper>1</implicitSpringDamper>
     </gazebo>

File: chapter06/baxter_camera/urdf/pedestal/pedestal.xacro (robot description, xacro)
@@ -2,8 +2,7 @@
 <robot name="pedistal" xmlns:xacro="http://www.ros.org/wiki/xacro">
   <!-- Arguments and Defaults-->
-  <xacro:arg name="gazebo" default="false"/>
   <link name="pedestal">
     <visual>
-      <origin rpy="0 0 0" xyz="0 0 0"/>
+      <origin rpy="0 0 0" xyz="0 0 0.93"/>
       <geometry>
         <mesh filename="package://baxter_camera/meshes/base/PEDESTAL.DAE"/>
@@ -14,7 +13,7 @@
     </visual>
     <collision>
-      <origin rpy="0 0 0" xyz="0 0 0"/>
+      <origin rpy="0 0 0" xyz="0 0 0.93"/>
       <geometry>
-        <mesh filename="package://baxter_camera/meshes/base/pedestal_link_collision.DAE"/>
+        <mesh filename="package://baxter_camera/meshes/base/PEDESTAL.STL"/>
       </geometry>
     </collision>
@@ -26,15 +25,13 @@
   </link>
   <joint name="pedestal_fixed" type="fixed">
-    <origin rpy="0 0 0" xyz="0.0 0.0 0.0"/>
-    <parent link="torso"/>
+    <origin rpy="0 0 0" xyz="0.0 0.0 0"/>
+    <parent link="base"/>
     <child link="pedestal"/>
   </joint>
-  <xacro:if value="$(arg gazebo)">
-    <!-- When using the pedistal, fix Baxter to Gazebo world with 'base' frame -->
-    <link name="world"/>
-    <joint name="fixed" type="fixed">
-      <parent link="world"/>
-      <child link="base"/>
-    </joint>
-  </xacro:if>
+  <link name="world"/>
+  <joint name="fixed" type="fixed">
+    <origin rpy="0 0 0" xyz="0.0 0.0 0"/>
+    <parent link="world"/>
+    <child link="base"/>
+  </joint>
 </robot>
